Commit message: Improve real grasping and update project

File: my_robot_description/urdf/arm.xacro (robot description, xacro)
@@ -57,14 +57,12 @@
     <link name="left_finger_link">
         <visual>
-            <origin xyz="0.04 0 0"
-                    rpy="0 0 0"/>
+            <origin xyz="0.04 0 0" rpy="0 0 0"/>
             <geometry>
-                <box size="0.08 0.01 0.02"/>
+                <box size="0.08 0.015 0.025"/>
             </geometry>
             <material name="gray"/>
         </visual>
         <collision>
-            <origin xyz="0.04 0.03 0"
-                    rpy="0 0 0"/>
+            <origin xyz="0.04 0 0" rpy="0 0 0"/>
             <geometry>
                 <box size="0.08 0.02 0.03"/>
@@ -72,28 +70,19 @@
         </collision>
         <inertial>
-            <origin xyz="0.04 0.03 0"
-                    rpy="0 0 0"/>
+            <origin xyz="0.04 0 0" rpy="0 0 0"/>
             <mass value="0.05"/>
-            <inertia
-                ixx="0.0001"
-                ixy="0"
-                ixz="0"
-                iyy="0.0001"
-                iyz="0"
-                izz="0.0001"/>
+            <inertia ixx="0.0001" ixy="0" ixz="0" iyy="0.0001" iyz="0" izz="0.0001"/>
         </inertial>
     </link>
     <link name="right_finger_link">
         <visual>
-            <origin xyz="0.04 0 0"
-                    rpy="0 0 0"/>
+            <origin xyz="0.04 0 0" rpy="0 0 0"/>
             <geometry>
-                <box size="0.08 0.01 0.02"/>
+                <box size="0.08 0.015 0.025"/>
             </geometry>
             <material name="gray"/>
         </visual>
         <collision>
-            <origin xyz="0.04 -0.03 0"
-                    rpy="0 0 0"/>
+            <origin xyz="0.04 0 0" rpy="0 0 0"/>
             <geometry>
                 <box size="0.08 0.02 0.03"/>
@@ -101,14 +90,7 @@
         </collision>
         <inertial>
-            <origin xyz="0.04 -0.03 0"
-                    rpy="0 0 0"/>
+            <origin xyz="0.04 0 0" rpy="0 0 0"/>
             <mass value="0.05"/>
-            <inertia
-                ixx="0.0001"
-                ixy="0"
-                ixz="0"
-                iyy="0.0001"
-                iyz="0"
-                izz="0.0001"/>
+            <inertia ixx="0.0001" ixy="0" ixz="0" iyy="0.0001" iyz="0" izz="0.0001"/>
         </inertial>
     </link>
@@ -172,7 +154,8 @@
         <limit
             lower="0"
-            upper="0.5"
-            effort="10"
-            velocity="1"/>
+            upper="0.6"
+            effort="20"
+            velocity="1.0"/>
+        <dynamics damping="2.0" friction="0.5"/>
     </joint>
     <joint name="right_finger_joint"
@@ -185,7 +168,8 @@
         <limit
             lower="0"
-            upper="0.5"
-            effort="10"
-            velocity="1"/>
+            upper="0.6"
+            effort="20"
+            velocity="1.0"/>
+        <dynamics damping="2.0" friction="0.5"/>
     </joint>
 </robot>

File: my_robot_description/urdf/mobile_base_gazebo.xacro (robot description, xacro)
@@ -14,10 +14,10 @@
     </gazebo>
     <gazebo reference="left_finger_link">
-        <mu1>5.0</mu1>
-        <mu2>5.0</mu2>
+        <mu1>10.0</mu1>
+        <mu2>10.0</mu2>
     </gazebo>
     <gazebo reference="right_finger_link">
-        <mu1>5.0</mu1>
-        <mu2>5.0</mu2>
+        <mu1>10.0</mu1>
+        <mu2>10.0</mu2>
     </gazebo>
     <gazebo>
@@ -53,5 +53,5 @@
             <joint_name>left_finger_joint</joint_name>
             <topic>/left_finger_joint/cmd_pos</topic>
-            <p_gain>10</p_gain>
+            <p_gain>30</p_gain>
         </plugin>
     </gazebo>
@@ -62,5 +62,5 @@
             <joint_name>right_finger_joint</joint_name>
             <topic>/right_finger_joint/cmd_pos</topic>
-            <p_gain>10</p_gain>
+            <p_gain>30</p_gain>
         </plugin>
     </gazebo>
@@ -83,5 +83,5 @@
         </plugin>
     </gazebo>
-    <gazebo>
+    <!-- <gazebo>
         <plugin
             filename="gz-sim-detachable-joint-system"
@@ -94,4 +94,4 @@
             <start_attached>false</start_attached>
         </plugin>
-    </gazebo>
+    </gazebo> -->
 </robot>
